File: Backplane/Backplane/Backplane.kicad_pcb (KiCad board)
At the start: 2 copper layers, 156.6 x 102.6 mm, 8 parts, among them J1 Conn_02x40_Counter_Clockwise, J2 Conn_02x40_Counter_Clockwise, J3 Conn_02x40_Counter_Clockwise, J4 Conn_02x40_Counter_Clockwise, J5 Conn_02x40_Counter_Clockwise, J6 Conn_02x40_Counter_Clockwise, J7 Conn_02x40_Counter_Clockwise, J8 Conn_02x40_Counter_Clockwise

Commit message: Final push to JLCPCB for latest rev
Parts:
- J8: footprint Connector_PinSocket_2.54mm:PinSocket_2x40_P2.54mm_Vertical -> Connector_PinHeader_2.54mm:PinHeader_2x40_P2.54mm_Horizontal
- moved J1 179.0 mm to (223.4, 142.9)
- moved J2 179.0 mm to (217.2, 142.9)
- moved J3 179.0 mm to (191.8, 142.9)
- moved J4 179.0 mm to (166.4, 142.9)
- moved J5 179.0 mm to (141.0, 142.9)
- moved J6 179.0 mm to (115.6, 142.9)
- moved J7 179.0 mm to (90.2, 142.9)
- moved J8 179.0 mm to (83.9, 142.9)
Connections:
- J1 pad 10: /10 -> /76
- J1 pad 11: /11 -> /6
- J1 pad 12: /12 -> /75
- J1 pad 13: /13 -> /7
- J1 pad 14: /14 -> /74
- J1 pad 15: /15 -> /8
- J1 pad 16: /16 -> /73
- J1 pad 17: /17 -> /9
- J1 pad 18: /18 -> /72
- J1 pad 19: /19 -> /10
- J1 pad 2: /2 -> /80
- J1 pad 20: /20 -> /71
- J1 pad 21: /21 -> /11
- J1 pad 22: /22 -> /70
- J1 pad 23: /23 -> /12
- J1 pad 24: /24 -> /69
- J1 pad 25: /25 -> /13
- J1 pad 26: /26 -> /68
- J1 pad 27: /27 -> /14
- J1 pad 28: /28 -> /67
- J1 pad 29: /29 -> /15
- J1 pad 3: /3 -> /2
- J1 pad 30: /30 -> /66
- J1 pad 31: /31 -> /16
- J1 pad 32: /32 -> /65
- J1 pad 33: /33 -> /17
- J1 pad 34: /34 -> /64
- J1 pad 35: /35 -> /18
- J1 pad 36: /36 -> /63
- J1 pad 37: /37 -> /19
- J1 pad 38: /38 -> /62
- J1 pad 39: /39 -> /20
- J1 pad 4: /4 -> /79
- J1 pad 40: /40 -> /61
- J1 pad 41: /41 -> /21
- J1 pad 42: /42 -> /60
- J1 pad 43: /43 -> /22
- J1 pad 44: /44 -> /59
- J1 pad 45: /45 -> /23
- J1 pad 46: /46 -> /58
- J1 pad 47: /47 -> /24
- J1 pad 48: /48 -> /57
- J1 pad 49: /49 -> /25
- J1 pad 5: /5 -> /3
- J1 pad 50: /50 -> /56
- J1 pad 51: /51 -> /26
- J1 pad 52: /52 -> /55
- J1 pad 53: /53 -> /27
- J1 pad 55: /55 -> /28
- J1 pad 56: /56 -> /53
- J1 pad 57: /57 -> /29
- J1 pad 58: /58 -> /52
- J1 pad 59: /59 -> /30
- J1 pad 6: /6 -> /78
- J1 pad 60: /60 -> /51
- J1 pad 61: /61 -> /31
- J1 pad 62: /62 -> /50
- J1 pad 63: /63 -> /32
- J1 pad 64: /64 -> /49
- J1 pad 65: /65 -> /33
- J1 pad 66: /66 -> /48
- J1 pad 67: /67 -> /34
- J1 pad 68: /68 -> /47
- J1 pad 69: /69 -> /35
- J1 pad 7: /7 -> /4
- J1 pad 70: /70 -> /46
- J1 pad 71: /71 -> /36
- J1 pad 72: /72 -> /45
- J1 pad 73: /73 -> /37
- J1 pad 74: /74 -> /44
- J1 pad 75: /75 -> /38
- J1 pad 76: /76 -> /43
- J1 pad 77: /77 -> /39
- J1 pad 78: /78 -> /42
- J1 pad 79: /79 -> /40
- J1 pad 8: /8 -> /77
- J1 pad 80: /80 -> /41
- J1 pad 9: /9 -> /5
- J2 pad 10: /10 -> /76
- J2 pad 11: /11 -> /6
- J2 pad 12: /12 -> /75
- J2 pad 13: /13 -> /7
- J2 pad 14: /14 -> /74
- J2 pad 15: /15 -> /8
- J2 pad 16: /16 -> /73
- J2 pad 17: /17 -> /9
- J2 pad 18: /18 -> /72
- J2 pad 19: /19 -> /10
- J2 pad 2: /2 -> /80
- J2 pad 20: /20 -> /71
- J2 pad 21: /21 -> /11
- J2 pad 22: /22 -> /70
- J2 pad 23: /23 -> /12
- J2 pad 24: /24 -> /69
- J2 pad 25: /25 -> /13
- J2 pad 26: /26 -> /68
- J2 pad 27: /27 -> /14
- J2 pad 28: /28 -> /67
- J2 pad 29: /29 -> /15
- J2 pad 3: /3 -> /2
- J2 pad 30: /30 -> /66
- J2 pad 31: /31 -> /16
- J2 pad 32: /32 -> /65
- J2 pad 33: /33 -> /17
- J2 pad 34: /34 -> /64
- J2 pad 35: /35 -> /18
- J2 pad 36: /36 -> /63
- J2 pad 37: /37 -> /19
- J2 pad 38: /38 -> /62
- J2 pad 39: /39 -> /20
- J2 pad 4: /4 -> /79
- J2 pad 40: /40 -> /61
- J2 pad 41: /41 -> /21
- J2 pad 42: /42 -> /60
- J2 pad 43: /43 -> /22
- J2 pad 44: /44 -> /59
- J2 pad 45: /45 -> /23
- J2 pad 46: /46 -> /58
- J2 pad 47: /47 -> /24
- J2 pad 48: /48 -> /57
- J2 pad 49: /49 -> /25
- J2 pad 5: /5 -> /3
- J2 pad 50: /50 -> /56
- J2 pad 51: /51 -> /26
- J2 pad 52: /52 -> /55
- J2 pad 53: /53 -> /27
- J2 pad 55: /55 -> /28
- J2 pad 56: /56 -> /53
- J2 pad 57: /57 -> /29
- J2 pad 58: /58 -> /52
- J2 pad 59: /59 -> /30
- J2 pad 6: /6 -> /78
- J2 pad 60: /60 -> /51
- J2 pad 61: /61 -> /31
- J2 pad 62: /62 -> /50
- J2 pad 63: /63 -> /32
- J2 pad 64: /64 -> /49
- J2 pad 65: /65 -> /33
- J2 pad 66: /66 -> /48
- J2 pad 67: /67 -> /34
- J2 pad 68: /68 -> /47
- J2 pad 69: /69 -> /35
- J2 pad 7: /7 -> /4
- J2 pad 70: /70 -> /46
- J2 pad 71: /71 -> /36
- J2 pad 72: /72 -> /45
- J2 pad 73: /73 -> /37
- J2 pad 74: /74 -> /44
- J2 pad 75: /75 -> /38
- J2 pad 76: /76 -> /43
- J2 pad 77: /77 -> /39
- J2 pad 78: /78 -> /42
- J2 pad 79: /79 -> /40
- J2 pad 8: /8 -> /77
- J2 pad 80: /80 -> /41
- J2 pad 9: /9 -> /5
- J3 pad 10: /10 -> /76
- J3 pad 11: /11 -> /6
- J3 pad 12: /12 -> /75
- J3 pad 13: /13 -> /7
- J3 pad 14: /14 -> /74
- J3 pad 15: /15 -> /8
- J3 pad 16: /16 -> /73
- J3 pad 17: /17 -> /9
- J3 pad 18: /18 -> /72
- J3 pad 19: /19 -> /10
- J3 pad 2: /2 -> /80
- J3 pad 20: /20 -> /71
- J3 pad 21: /21 -> /11
- J3 pad 22: /22 -> /70
- J3 pad 23: /23 -> /12
- J3 pad 24: /24 -> /69
- J3 pad 25: /25 -> /13
- J3 pad 26: /26 -> /68
- J3 pad 27: /27 -> /14
- J3 pad 28: /28 -> /67
- J3 pad 29: /29 -> /15
- J3 pad 3: /3 -> /2
- J3 pad 30: /30 -> /66
- J3 pad 31: /31 -> /16
- J3 pad 32: /32 -> /65
- J3 pad 33: /33 -> /17
- J3 pad 34: /34 -> /64
- J3 pad 35: /35 -> /18
- J3 pad 36: /36 -> /63
- J3 pad 37: /37 -> /19
- J3 pad 38: /38 -> /62
- J3 pad 39: /39 -> /20
- J3 pad 4: /4 -> /79
- J3 pad 40: /40 -> /61
- J3 pad 41: /41 -> /21
- J3 pad 42: /42 -> /60
- J3 pad 43: /43 -> /22
- J3 pad 44: /44 -> /59
- J3 pad 45: /45 -> /23
- J3 pad 46: /46 -> /58
- J3 pad 47: /47 -> /24
- J3 pad 48: /48 -> /57
- J3 pad 49: /49 -> /25
- J3 pad 5: /5 -> /3
- J3 pad 50: /50 -> /56
- J3 pad 51: /51 -> /26
- J3 pad 52: /52 -> /55
- J3 pad 53: /53 -> /27
- J3 pad 55: /55 -> /28
- J3 pad 56: /56 -> /53
- J3 pad 57: /57 -> /29
- J3 pad 58: /58 -> /52
- J3 pad 59: /59 -> /30
- J3 pad 6: /6 -> /78
- J3 pad 60: /60 -> /51
- J3 pad 61: /61 -> /31
- J3 pad 62: /62 -> /50
- J3 pad 63: /63 -> /32
- J3 pad 64: /64 -> /49
- J3 pad 65: /65 -> /33
- J3 pad 66: /66 -> /48
- J3 pad 67: /67 -> /34
- J3 pad 68: /68 -> /47
- J3 pad 69: /69 -> /35
- J3 pad 7: /7 -> /4
- J3 pad 70: /70 -> /46
- J3 pad 71: /71 -> /36
- J3 pad 72: /72 -> /45
- J3 pad 73: /73 -> /37
- J3 pad 74: /74 -> /44
- J3 pad 75: /75 -> /38
- J3 pad 76: /76 -> /43
- J3 pad 77: /77 -> /39
- J3 pad 78: /78 -> /42
- J3 pad 79: /79 -> /40
- J3 pad 8: /8 -> /77
- J3 pad 80: /80 -> /41
- J3 pad 9: /9 -> /5
- J4 pad 10: /10 -> /76
- J4 pad 11: /11 -> /6
- J4 pad 12: /12 -> /75
- J4 pad 13: /13 -> /7
- J4 pad 14: /14 -> /74
- J4 pad 15: /15 -> /8
- J4 pad 16: /16 -> /73
- J4 pad 17: /17 -> /9
- J4 pad 18: /18 -> /72
- J4 pad 19: /19 -> /10
- J4 pad 2: /2 -> /80
- J4 pad 20: /20 -> /71
- J4 pad 21: /21 -> /11
- J4 pad 22: /22 -> /70
- J4 pad 23: /23 -> /12
- J4 pad 24: /24 -> /69
- J4 pad 25: /25 -> /13
- J4 pad 26: /26 -> /68
- J4 pad 27: /27 -> /14
- J4 pad 28: /28 -> /67
- J4 pad 29: /29 -> /15
- J4 pad 3: /3 -> /2
- J4 pad 30: /30 -> /66
- J4 pad 31: /31 -> /16
- J4 pad 32: /32 -> /65
- J4 pad 33: /33 -> /17
- J4 pad 34: /34 -> /64
- J4 pad 35: /35 -> /18
- J4 pad 36: /36 -> /63
- J4 pad 37: /37 -> /19
- J4 pad 38: /38 -> /62
- J4 pad 39: /39 -> /20
- J4 pad 4: /4 -> /79
- J4 pad 40: /40 -> /61
- J4 pad 41: /41 -> /21
- J4 pad 42: /42 -> /60
- J4 pad 43: /43 -> /22
- J4 pad 44: /44 -> /59
- J4 pad 45: /45 -> /23
- J4 pad 46: /46 -> /58
- J4 pad 47: /47 -> /24
- J4 pad 48: /48 -> /57
- J4 pad 49: /49 -> /25
- J4 pad 5: /5 -> /3
- J4 pad 50: /50 -> /56
- J4 pad 51: /51 -> /26
- J4 pad 52: /52 -> /55
- J4 pad 53: /53 -> /27
- J4 pad 55: /55 -> /28
- J4 pad 56: /56 -> /53
- J4 pad 57: /57 -> /29
- J4 pad 58: /58 -> /52
- J4 pad 59: /59 -> /30
- J4 pad 6: /6 -> /78
- J4 pad 60: /60 -> /51
- J4 pad 61: /61 -> /31
- J4 pad 62: /62 -> /50
- J4 pad 63: /63 -> /32
- J4 pad 64: /64 -> /49
- J4 pad 65: /65 -> /33
- J4 pad 66: /66 -> /48
- J4 pad 67: /67 -> /34
- J4 pad 68: /68 -> /47
- J4 pad 69: /69 -> /35
- J4 pad 7: /7 -> /4
- J4 pad 70: /70 -> /46
- J4 pad 71: /71 -> /36
- J4 pad 72: /72 -> /45
- J4 pad 73: /73 -> /37
- J4 pad 74: /74 -> /44
- J4 pad 75: /75 -> /38
- J4 pad 76: /76 -> /43
- J4 pad 77: /77 -> /39
- J4 pad 78: /78 -> /42
- J4 pad 79: /79 -> /40
- J4 pad 8: /8 -> /77
- J4 pad 80: /80 -> /41
- J4 pad 9: /9 -> /5
- J5 pad 10: /10 -> /76
- J5 pad 11: /11 -> /6
- J5 pad 12: /12 -> /75
- J5 pad 13: /13 -> /7
- J5 pad 14: /14 -> /74
- J5 pad 15: /15 -> /8
- J5 pad 16: /16 -> /73
- J5 pad 17: /17 -> /9
- J5 pad 18: /18 -> /72
- J5 pad 19: /19 -> /10
- J5 pad 2: /2 -> /80
- J5 pad 20: /20 -> /71
- J5 pad 21: /21 -> /11
- J5 pad 22: /22 -> /70
- J5 pad 23: /23 -> /12
- J5 pad 24: /24 -> /69
- J5 pad 25: /25 -> /13
- J5 pad 26: /26 -> /68
- J5 pad 27: /27 -> /14
- J5 pad 28: /28 -> /67
- J5 pad 29: /29 -> /15
- J5 pad 3: /3 -> /2
- J5 pad 30: /30 -> /66
- J5 pad 31: /31 -> /16
- J5 pad 32: /32 -> /65
- J5 pad 33: /33 -> /17
- J5 pad 34: /34 -> /64
- J5 pad 35: /35 -> /18
- J5 pad 36: /36 -> /63
- J5 pad 37: /37 -> /19
- J5 pad 38: /38 -> /62
- J5 pad 39: /39 -> /20
- J5 pad 4: /4 -> /79
- J5 pad 40: /40 -> /61
- J5 pad 41: /41 -> /21
- J5 pad 42: /42 -> /60
- J5 pad 43: /43 -> /22
- J5 pad 44: /44 -> /59
- J5 pad 45: /45 -> /23
- J5 pad 46: /46 -> /58
- J5 pad 47: /47 -> /24
- J5 pad 48: /48 -> /57
- J5 pad 49: /49 -> /25
- J5 pad 5: /5 -> /3
- J5 pad 50: /50 -> /56
- J5 pad 51: /51 -> /26
- J5 pad 52: /52 -> /55
- J5 pad 53: /53 -> /27
- J5 pad 55: /55 -> /28
- J5 pad 56: /56 -> /53
- J5 pad 57: /57 -> /29
- J5 pad 58: /58 -> /52
- J5 pad 59: /59 -> /30
- J5 pad 6: /6 -> /78
- J5 pad 60: /60 -> /51
- J5 pad 61: /61 -> /31
- J5 pad 62: /62 -> /50
- J5 pad 63: /63 -> /32
- J5 pad 64: /64 -> /49
- J5 pad 65: /65 -> /33
- J5 pad 66: /66 -> /48
- J5 pad 67: /67 -> /34
- J5 pad 68: /68 -> /47
- J5 pad 69: /69 -> /35
- J5 pad 7: /7 -> /4
- J5 pad 70: /70 -> /46
- J5 pad 71: /71 -> /36
- J5 pad 72: /72 -> /45
- J5 pad 73: /73 -> /37
- J5 pad 74: /74 -> /44
- J5 pad 75: /75 -> /38
- J5 pad 76: /76 -> /43
- J5 pad 77: /77 -> /39
- J5 pad 78: /78 -> /42
- J5 pad 79: /79 -> /40
- J5 pad 8: /8 -> /77
- J5 pad 80: /80 -> /41
- J5 pad 9: /9 -> /5
- J6 pad 10: /10 -> /76
- J6 pad 11: /11 -> /6
- J6 pad 12: /12 -> /75
- J6 pad 13: /13 -> /7
- J6 pad 14: /14 -> /74
- J6 pad 15: /15 -> /8
- J6 pad 16: /16 -> /73
- J6 pad 17: /17 -> /9
- J6 pad 18: /18 -> /72
- J6 pad 19: /19 -> /10
- J6 pad 2: /2 -> /80
- J6 pad 20: /20 -> /71
- J6 pad 21: /21 -> /11
- J6 pad 22: /22 -> /70
- J6 pad 23: /23 -> /12
- J6 pad 24: /24 -> /69
- J6 pad 25: /25 -> /13
- J6 pad 26: /26 -> /68
- J6 pad 27: /27 -> /14
- J6 pad 28: /28 -> /67
- J6 pad 29: /29 -> /15
- J6 pad 3: /3 -> /2
- J6 pad 30: /30 -> /66
- J6 pad 31: /31 -> /16
- J6 pad 32: /32 -> /65
- J6 pad 33: /33 -> /17
- J6 pad 34: /34 -> /64
- J6 pad 35: /35 -> /18
- J6 pad 36: /36 -> /63
- J6 pad 37: /37 -> /19
- J6 pad 38: /38 -> /62
- J6 pad 39: /39 -> /20
- J6 pad 4: /4 -> /79
- J6 pad 40: /40 -> /61
- J6 pad 41: /41 -> /21
- J6 pad 42: /42 -> /60
- J6 pad 43: /43 -> /22
- J6 pad 44: /44 -> /59
- J6 pad 45: /45 -> /23
- J6 pad 46: /46 -> /58
- J6 pad 47: /47 -> /24
- J6 pad 48: /48 -> /57
- J6 pad 49: /49 -> /25
- J6 pad 5: /5 -> /3
- J6 pad 50: /50 -> /56
- J6 pad 51: /51 -> /26
- J6 pad 52: /52 -> /55
- J6 pad 53: /53 -> /27
- J6 pad 55: /55 -> /28
- J6 pad 56: /56 -> /53
- J6 pad 57: /57 -> /29
- J6 pad 58: /58 -> /52
- J6 pad 59: /59 -> /30
- J6 pad 6: /6 -> /78
- J6 pad 60: /60 -> /51
- J6 pad 61: /61 -> /31
- J6 pad 62: /62 -> /50
- J6 pad 63: /63 -> /32
- J6 pad 64: /64 -> /49
- J6 pad 65: /65 -> /33
- J6 pad 66: /66 -> /48
- J6 pad 67: /67 -> /34
- J6 pad 68: /68 -> /47
- J6 pad 69: /69 -> /35
- J6 pad 7: /7 -> /4
- J6 pad 70: /70 -> /46
- J6 pad 71: /71 -> /36
- J6 pad 72: /72 -> /45
- J6 pad 73: /73 -> /37
- J6 pad 74: /74 -> /44
- J6 pad 75: /75 -> /38
- J6 pad 76: /76 -> /43
- J6 pad 77: /77 -> /39
- J6 pad 78: /78 -> /42
- J6 pad 79: /79 -> /40
- J6 pad 8: /8 -> /77
- J6 pad 80: /80 -> /41
- J6 pad 9: /9 -> /5
- J7 pad 10: /10 -> /76
- J7 pad 11: /11 -> /6
- J7 pad 12: /12 -> /75
- J7 pad 13: /13 -> /7
- J7 pad 14: /14 -> /74
- J7 pad 15: /15 -> /8
- J7 pad 16: /16 -> /73
- J7 pad 17: /17 -> /9
- J7 pad 18: /18 -> /72
- J7 pad 19: /19 -> /10
- J7 pad 2: /2 -> /80
- J7 pad 20: /20 -> /71
- J7 pad 21: /21 -> /11
- J7 pad 22: /22 -> /70
- J7 pad 23: /23 -> /12
- J7 pad 24: /24 -> /69
- J7 pad 25: /25 -> /13
- J7 pad 26: /26 -> /68
- J7 pad 27: /27 -> /14
- J7 pad 28: /28 -> /67
- J7 pad 29: /29 -> /15
- J7 pad 3: /3 -> /2
- J7 pad 30: /30 -> /66
- J7 pad 31: /31 -> /16
- J7 pad 32: /32 -> /65
- J7 pad 33: /33 -> /17
- J7 pad 34: /34 -> /64
- J7 pad 35: /35 -> /18
- J7 pad 36: /36 -> /63
- J7 pad 37: /37 -> /19
- J7 pad 38: /38 -> /62
- J7 pad 39: /39 -> /20
- J7 pad 4: /4 -> /79
- J7 pad 40: /40 -> /61
- J7 pad 41: /41 -> /21
- J7 pad 42: /42 -> /60
- J7 pad 43: /43 -> /22
- J7 pad 44: /44 -> /59
- J7 pad 45: /45 -> /23
- J7 pad 46: /46 -> /58
- J7 pad 47: /47 -> /24
- J7 pad 48: /48 -> /57
- J7 pad 49: /49 -> /25
- J7 pad 5: /5 -> /3
- J7 pad 50: /50 -> /56
- J7 pad 51: /51 -> /26
- J7 pad 52: /52 -> /55
- J7 pad 53: /53 -> /27
- J7 pad 55: /55 -> /28
- J7 pad 56: /56 -> /53
- J7 pad 57: /57 -> /29
- J7 pad 58: /58 -> /52
- J7 pad 59: /59 -> /30
- J7 pad 6: /6 -> /78
- J7 pad 60: /60 -> /51
- J7 pad 61: /61 -> /31
- J7 pad 62: /62 -> /50
- J7 pad 63: /63 -> /32
- J7 pad 64: /64 -> /49
- J7 pad 65: /65 -> /33
- J7 pad 66: /66 -> /48
- J7 pad 67: /67 -> /34
- J7 pad 68: /68 -> /47
- J7 pad 69: /69 -> /35
- J7 pad 7: /7 -> /4
- J7 pad 70: /70 -> /46
- J7 pad 71: /71 -> /36
- J7 pad 72: /72 -> /45
- J7 pad 73: /73 -> /37
- J7 pad 74: /74 -> /44
- J7 pad 75: /75 -> /38
- J7 pad 76: /76 -> /43
- J7 pad 77: /77 -> /39
- J7 pad 78: /78 -> /42
- J7 pad 79: /79 -> /40
- J7 pad 8: /8 -> /77
- J7 pad 80: /80 -> /41
- J7 pad 9: /9 -> /5
- J8 pad 10: /10 -> /76
- J8 pad 11: /11 -> /6
- J8 pad 12: /12 -> /75
- J8 pad 13: /13 -> /7
- J8 pad 14: /14 -> /74
- J8 pad 15: /15 -> /8
- J8 pad 16: /16 -> /73
- J8 pad 17: /17 -> /9
- J8 pad 18: /18 -> /72
- J8 pad 19: /19 -> /10
- J8 pad 2: /2 -> /80
- J8 pad 20: /20 -> /71
- J8 pad 21: /21 -> /11
- J8 pad 22: /22 -> /70
- J8 pad 23: /23 -> /12
- J8 pad 24: /24 -> /69
- J8 pad 25: /25 -> /13
- J8 pad 26: /26 -> /68
- J8 pad 27: /27 -> /14
- J8 pad 28: /28 -> /67
- J8 pad 29: /29 -> /15
- J8 pad 3: /3 -> /2
- J8 pad 30: /30 -> /66
- J8 pad 31: /31 -> /16
- J8 pad 32: /32 -> /65
- J8 pad 33: /33 -> /17
- J8 pad 34: /34 -> /64
- J8 pad 35: /35 -> /18
- J8 pad 36: /36 -> /63
- J8 pad 37: /37 -> /19
- J8 pad 38: /38 -> /62
- J8 pad 39: /39 -> /20
- J8 pad 4: /4 -> /79
- J8 pad 40: /40 -> /61
- J8 pad 41: /41 -> /21
- J8 pad 42: /42 -> /60
- J8 pad 43: /43 -> /22
- J8 pad 44: /44 -> /59
- J8 pad 45: /45 -> /23
- J8 pad 46: /46 -> /58
- J8 pad 47: /47 -> /24
- J8 pad 48: /48 -> /57
- J8 pad 49: /49 -> /25
- J8 pad 5: /5 -> /3
- J8 pad 50: /50 -> /56
- J8 pad 51: /51 -> /26
- J8 pad 52: /52 -> /55
- J8 pad 53: /53 -> /27
- J8 pad 55: /55 -> /28
- J8 pad 56: /56 -> /53
- J8 pad 57: /57 -> /29
- J8 pad 58: /58 -> /52
- J8 pad 59: /59 -> /30
- J8 pad 6: /6 -> /78
- J8 pad 60: /60 -> /51
- J8 pad 61: /61 -> /31
- J8 pad 62: /62 -> /50
- J8 pad 63: /63 -> /32
- J8 pad 64: /64 -> /49
- J8 pad 65: /65 -> /33
- J8 pad 66: /66 -> /48
- J8 pad 67: /67 -> /34
- J8 pad 68: /68 -> /47
- J8 pad 69: /69 -> /35
- J8 pad 7: /7 -> /4
- J8 pad 70: /70 -> /46
- J8 pad 71: /71 -> /36
- J8 pad 72: /72 -> /45
- J8 pad 73: /73 -> /37
- J8 pad 74: /74 -> /44
- J8 pad 75: /75 -> /38
- J8 pad 76: /76 -> /43
- J8 pad 77: /77 -> /39
- J8 pad 78: /78 -> /42
- J8 pad 79: /79 -> /40
- J8 pad 8: /8 -> /77
- J8 pad 80: /80 -> /41
- J8 pad 9: /9 -> /5
Routing:
- net /80: track 147.6 -> 161.5 mm
- net /71: track 146.3 -> 154.9 mm
- net /75: track 146.3 -> 153.6 mm
- net /79: track 146.4 -> 153.6 mm
- net /78: track 146.3 -> 152.6 mm
- net /70: track 146.3 -> 152.0 mm
- net /73: track 146.4 -> 152.0 mm
- net /72: track 146.6 -> 152.0 mm
- net /45: track 146.3 -> 151.7 mm
- net /56: track 146.3 -> 151.5 mm
- net /60: track 146.3 -> 151.5 mm
- net /51: track 146.3 -> 151.5 mm
- net /50: track 146.4 -> 151.7 mm
- net /47: track 146.3 -> 151.5 mm
- net /57: track 146.3 -> 151.5 mm
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Other:
- board size 156.6 x 102.6 mm -> 158.8 x 102.6 mm
- net class Default: trace_width 0.35 -> 0.25
- net class POWER: trace_width 0.5 -> 0.25
