File: Backplane/Backplane/Backplane.sch (KiCad schematic (older format))
At the start: 8 parts, among them J1 Conn_02x40_Counter_Clockwise, J2 Conn_02x40_Counter_Clockwise, J3 Conn_02x40_Counter_Clockwise, J4 Conn_02x40_Counter_Clockwise, J5 Conn_02x40_Counter_Clockwise, J6 Conn_02x40_Counter_Clockwise, J7 Conn_02x40_Counter_Clockwise, J8 Conn_02x40_Counter_Clockwise

Commit message: Final push to JLCPCB for latest rev
Parts:
- J1, J2, J3, J4, J5, J6, J7, J8: symbol Connector_Generic:Conn_02x40_Counter_Clockwise -> Connector_Generic:Conn_02x40_Odd_Even
Connections:
- net 10: now also J1.19 (Pin_19), J2.19 (Pin_19), J3.19 (Pin_19), J4.19 (Pin_19), J5.19 (Pin_19), J6.19 (Pin_19), J7.19 (Pin_19), J8.19 (Pin_19); no longer J1.10 (Pin_10), J2.10 (Pin_10), J3.10 (Pin_10), J4.10 (Pin_10), J5.10 (Pin_10), J6.10 (Pin_10), J7.10 (Pin_10), J8.10 (Pin_10)
- net 11: now also J1.21 (Pin_21), J2.21 (Pin_21), J3.21 (Pin_21), J4.21 (Pin_21), J5.21 (Pin_21), J6.21 (Pin_21), J7.21 (Pin_21), J8.21 (Pin_21); no longer J1.11 (Pin_11), J2.11 (Pin_11), J3.11 (Pin_11), J4.11 (Pin_11), J5.11 (Pin_11), J6.11 (Pin_11), J7.11 (Pin_11), J8.11 (Pin_11)
- net 12: now also J1.23 (Pin_23), J2.23 (Pin_23), J3.23 (Pin_23), J4.23 (Pin_23), J5.23 (Pin_23), J6.23 (Pin_23), J7.23 (Pin_23), J8.23 (Pin_23); no longer J1.12 (Pin_12), J2.12 (Pin_12), J3.12 (Pin_12), J4.12 (Pin_12), J5.12 (Pin_12), J6.12 (Pin_12), J7.12 (Pin_12), J8.12 (Pin_12)
- net 13: now also J1.25 (Pin_25), J2.25 (Pin_25), J3.25 (Pin_25), J4.25 (Pin_25), J5.25 (Pin_25), J6.25 (Pin_25), J7.25 (Pin_25), J8.25 (Pin_25); no longer J1.13 (Pin_13), J2.13 (Pin_13), J3.13 (Pin_13), J4.13 (Pin_13), J5.13 (Pin_13), J6.13 (Pin_13), J7.13 (Pin_13), J8.13 (Pin_13)
- net 14: now also J1.27 (Pin_27), J2.27 (Pin_27), J3.27 (Pin_27), J4.27 (Pin_27), J5.27 (Pin_27), J6.27 (Pin_27), J7.27 (Pin_27), J8.27 (Pin_27); no longer J1.14 (Pin_14), J2.14 (Pin_14), J3.14 (Pin_14), J4.14 (Pin_14), J5.14 (Pin_14), J6.14 (Pin_14), J7.14 (Pin_14), J8.14 (Pin_14)
- net 15: now also J1.29 (Pin_29), J2.29 (Pin_29), J3.29 (Pin_29), J4.29 (Pin_29), J5.29 (Pin_29), J6.29 (Pin_29), J7.29 (Pin_29), J8.29 (Pin_29); no longer J1.15 (Pin_15), J2.15 (Pin_15), J3.15 (Pin_15), J4.15 (Pin_15), J5.15 (Pin_15), J6.15 (Pin_15), J7.15 (Pin_15), J8.15 (Pin_15)
- net 16: now also J1.31 (Pin_31), J2.31 (Pin_31), J3.31 (Pin_31), J4.31 (Pin_31), J5.31 (Pin_31), J6.31 (Pin_31), J7.31 (Pin_31), J8.31 (Pin_31); no longer J1.16 (Pin_16), J2.16 (Pin_16), J3.16 (Pin_16), J4.16 (Pin_16), J5.16 (Pin_16), J6.16 (Pin_16), J7.16 (Pin_16), J8.16 (Pin_16)
- net 17: now also J1.33 (Pin_33), J2.33 (Pin_33), J3.33 (Pin_33), J4.33 (Pin_33), J5.33 (Pin_33), J6.33 (Pin_33), J7.33 (Pin_33), J8.33 (Pin_33); no longer J1.17 (Pin_17), J2.17 (Pin_17), J3.17 (Pin_17), J4.17 (Pin_17), J5.17 (Pin_17), J6.17 (Pin_17), J7.17 (Pin_17), J8.17 (Pin_17)
- net 18: now also J1.35 (Pin_35), J2.35 (Pin_35), J3.35 (Pin_35), J4.35 (Pin_35), J5.35 (Pin_35), J6.35 (Pin_35), J7.35 (Pin_35), J8.35 (Pin_35); no longer J1.18 (Pin_18), J2.18 (Pin_18), J3.18 (Pin_18), J4.18 (Pin_18), J5.18 (Pin_18), J6.18 (Pin_18), J7.18 (Pin_18), J8.18 (Pin_18)
- net 19: now also J1.37 (Pin_37), J2.37 (Pin_37), J3.37 (Pin_37), J4.37 (Pin_37), J5.37 (Pin_37), J6.37 (Pin_37), J7.37 (Pin_37), J8.37 (Pin_37); no longer J1.19 (Pin_19), J2.19 (Pin_19), J3.19 (Pin_19), J4.19 (Pin_19), J5.19 (Pin_19), J6.19 (Pin_19), J7.19 (Pin_19), J8.19 (Pin_19)
- net 2: now also J1.3 (Pin_3), J2.3 (Pin_3), J3.3 (Pin_3), J4.3 (Pin_3), J5.3 (Pin_3), J6.3 (Pin_3), J7.3 (Pin_3), J8.3 (Pin_3); no longer J1.2 (Pin_2), J2.2 (Pin_2), J3.2 (Pin_2), J4.2 (Pin_2), J5.2 (Pin_2), J6.2 (Pin_2), J7.2 (Pin_2), J8.2 (Pin_2)
- net 20: now also J1.39 (Pin_39), J2.39 (Pin_39), J3.39 (Pin_39), J4.39 (Pin_39), J5.39 (Pin_39), J6.39 (Pin_39), J7.39 (Pin_39), J8.39 (Pin_39); no longer J1.20 (Pin_20), J2.20 (Pin_20), J3.20 (Pin_20), J4.20 (Pin_20), J5.20 (Pin_20), J6.20 (Pin_20), J7.20 (Pin_20), J8.20 (Pin_20)
- net 21: now also J1.41 (Pin_41), J2.41 (Pin_41), J3.41 (Pin_41), J4.41 (Pin_41), J5.41 (Pin_41), J6.41 (Pin_41), J7.41 (Pin_41), J8.41 (Pin_41); no longer J1.21 (Pin_21), J2.21 (Pin_21), J3.21 (Pin_21), J4.21 (Pin_21), J5.21 (Pin_21), J6.21 (Pin_21), J7.21 (Pin_21), J8.21 (Pin_21)
- net 22: now also J1.43 (Pin_43), J2.43 (Pin_43), J3.43 (Pin_43), J4.43 (Pin_43), J5.43 (Pin_43), J6.43 (Pin_43), J7.43 (Pin_43), J8.43 (Pin_43); no longer J1.22 (Pin_22), J2.22 (Pin_22), J3.22 (Pin_22), J4.22 (Pin_22), J5.22 (Pin_22), J6.22 (Pin_22), J7.22 (Pin_22), J8.22 (Pin_22)
- net 23: now also J1.45 (Pin_45), J2.45 (Pin_45), J3.45 (Pin_45), J4.45 (Pin_45), J5.45 (Pin_45), J6.45 (Pin_45), J7.45 (Pin_45), J8.45 (Pin_45); no longer J1.23 (Pin_23), J2.23 (Pin_23), J3.23 (Pin_23), J4.23 (Pin_23), J5.23 (Pin_23), J6.23 (Pin_23), J7.23 (Pin_23), J8.23 (Pin_23)
- net 24: now also J1.47 (Pin_47), J2.47 (Pin_47), J3.47 (Pin_47), J4.47 (Pin_47), J5.47 (Pin_47), J6.47 (Pin_47), J7.47 (Pin_47), J8.47 (Pin_47); no longer J1.24 (Pin_24), J2.24 (Pin_24), J3.24 (Pin_24), J4.24 (Pin_24), J5.24 (Pin_24), J6.24 (Pin_24), J7.24 (Pin_24), J8.24 (Pin_24)
- net 25: now also J1.49 (Pin_49), J2.49 (Pin_49), J3.49 (Pin_49), J4.49 (Pin_49), J5.49 (Pin_49), J6.49 (Pin_49), J7.49 (Pin_49), J8.49 (Pin_49); no longer J1.25 (Pin_25), J2.25 (Pin_25), J3.25 (Pin_25), J4.25 (Pin_25), J5.25 (Pin_25), J6.25 (Pin_25), J7.25 (Pin_25), J8.25 (Pin_25)
- net 26: now also J1.51 (Pin_51), J2.51 (Pin_51), J3.51 (Pin_51), J4.51 (Pin_51), J5.51 (Pin_51), J6.51 (Pin_51), J7.51 (Pin_51), J8.51 (Pin_51); no longer J1.26 (Pin_26), J2.26 (Pin_26), J3.26 (Pin_26), J4.26 (Pin_26), J5.26 (Pin_26), J6.26 (Pin_26), J7.26 (Pin_26), J8.26 (Pin_26)
- net 27: now also J1.53 (Pin_53), J2.53 (Pin_53), J3.53 (Pin_53), J4.53 (Pin_53), J5.53 (Pin_53), J6.53 (Pin_53), J7.53 (Pin_53), J8.53 (Pin_53); no longer J1.27 (Pin_27), J2.27 (Pin_27), J3.27 (Pin_27), J4.27 (Pin_27), J5.27 (Pin_27), J6.27 (Pin_27), J7.27 (Pin_27), J8.27 (Pin_27)
- net 28: now also J1.55 (Pin_55), J2.55 (Pin_55), J3.55 (Pin_55), J4.55 (Pin_55), J5.55 (Pin_55), J6.55 (Pin_55), J7.55 (Pin_55), J8.55 (Pin_55); no longer J1.28 (Pin_28), J2.28 (Pin_28), J3.28 (Pin_28), J4.28 (Pin_28), J5.28 (Pin_28), J6.28 (Pin_28), J7.28 (Pin_28), J8.28 (Pin_28)
- net 29: now also J1.57 (Pin_57), J2.57 (Pin_57), J3.57 (Pin_57), J4.57 (Pin_57), J5.57 (Pin_57), J6.57 (Pin_57), J7.57 (Pin_57), J8.57 (Pin_57); no longer J1.29 (Pin_29), J2.29 (Pin_29), J3.29 (Pin_29), J4.29 (Pin_29), J5.29 (Pin_29), J6.29 (Pin_29), J7.29 (Pin_29), J8.29 (Pin_29)
- net 3: now also J1.5 (Pin_5), J2.5 (Pin_5), J3.5 (Pin_5), J4.5 (Pin_5), J5.5 (Pin_5), J6.5 (Pin_5), J7.5 (Pin_5), J8.5 (Pin_5); no longer J1.3 (Pin_3), J2.3 (Pin_3), J3.3 (Pin_3), J4.3 (Pin_3), J5.3 (Pin_3), J6.3 (Pin_3), J7.3 (Pin_3), J8.3 (Pin_3)
- net 30: now also J1.59 (Pin_59), J2.59 (Pin_59), J3.59 (Pin_59), J4.59 (Pin_59), J5.59 (Pin_59), J6.59 (Pin_59), J7.59 (Pin_59), J8.59 (Pin_59); no longer J1.30 (Pin_30), J2.30 (Pin_30), J3.30 (Pin_30), J4.30 (Pin_30), J5.30 (Pin_30), J6.30 (Pin_30), J7.30 (Pin_30), J8.30 (Pin_30)
- net 31: now also J1.61 (Pin_61), J2.61 (Pin_61), J3.61 (Pin_61), J4.61 (Pin_61), J5.61 (Pin_61), J6.61 (Pin_61), J7.61 (Pin_61), J8.61 (Pin_61); no longer J1.31 (Pin_31), J2.31 (Pin_31), J3.31 (Pin_31), J4.31 (Pin_31), J5.31 (Pin_31), J6.31 (Pin_31), J7.31 (Pin_31), J8.31 (Pin_31)
- net 32: now also J1.63 (Pin_63), J2.63 (Pin_63), J3.63 (Pin_63), J4.63 (Pin_63), J5.63 (Pin_63), J6.63 (Pin_63), J7.63 (Pin_63), J8.63 (Pin_63); no longer J1.32 (Pin_32), J2.32 (Pin_32), J3.32 (Pin_32), J4.32 (Pin_32), J5.32 (Pin_32), J6.32 (Pin_32), J7.32 (Pin_32), J8.32 (Pin_32)
- net 33: now also J1.65 (Pin_65), J2.65 (Pin_65), J3.65 (Pin_65), J4.65 (Pin_65), J5.65 (Pin_65), J6.65 (Pin_65), J7.65 (Pin_65), J8.65 (Pin_65); no longer J1.33 (Pin_33), J2.33 (Pin_33), J3.33 (Pin_33), J4.33 (Pin_33), J5.33 (Pin_33), J6.33 (Pin_33), J7.33 (Pin_33), J8.33 (Pin_33)
- net 34: now also J1.67 (Pin_67), J2.67 (Pin_67), J3.67 (Pin_67), J4.67 (Pin_67), J5.67 (Pin_67), J6.67 (Pin_67), J7.67 (Pin_67), J8.67 (Pin_67); no longer J1.34 (Pin_34), J2.34 (Pin_34), J3.34 (Pin_34), J4.34 (Pin_34), J5.34 (Pin_34), J6.34 (Pin_34), J7.34 (Pin_34), J8.34 (Pin_34)
- net 35: now also J1.69 (Pin_69), J2.69 (Pin_69), J3.69 (Pin_69), J4.69 (Pin_69), J5.69 (Pin_69), J6.69 (Pin_69), J7.69 (Pin_69), J8.69 (Pin_69); no longer J1.35 (Pin_35), J2.35 (Pin_35), J3.35 (Pin_35), J4.35 (Pin_35), J5.35 (Pin_35), J6.35 (Pin_35), J7.35 (Pin_35), J8.35 (Pin_35)
- net 36: now also J1.71 (Pin_71), J2.71 (Pin_71), J3.71 (Pin_71), J4.71 (Pin_71), J5.71 (Pin_71), J6.71 (Pin_71), J7.71 (Pin_71), J8.71 (Pin_71); no longer J1.36 (Pin_36), J2.36 (Pin_36), J3.36 (Pin_36), J4.36 (Pin_36), J5.36 (Pin_36), J6.36 (Pin_36), J7.36 (Pin_36), J8.36 (Pin_36)
- net 37: now also J1.73 (Pin_73), J2.73 (Pin_73), J3.73 (Pin_73), J4.73 (Pin_73), J5.73 (Pin_73), J6.73 (Pin_73), J7.73 (Pin_73), J8.73 (Pin_73); no longer J1.37 (Pin_37), J2.37 (Pin_37), J3.37 (Pin_37), J4.37 (Pin_37), J5.37 (Pin_37), J6.37 (Pin_37), J7.37 (Pin_37), J8.37 (Pin_37)
- net 38: now also J1.75 (Pin_75), J2.75 (Pin_75), J3.75 (Pin_75), J4.75 (Pin_75), J5.75 (Pin_75), J6.75 (Pin_75), J7.75 (Pin_75), J8.75 (Pin_75); no longer J1.38 (Pin_38), J2.38 (Pin_38), J3.38 (Pin_38), J4.38 (Pin_38), J5.38 (Pin_38), J6.38 (Pin_38), J7.38 (Pin_38), J8.38 (Pin_38)
- net 39: now also J1.77 (Pin_77), J2.77 (Pin_77), J3.77 (Pin_77), J4.77 (Pin_77), J5.77 (Pin_77), J6.77 (Pin_77), J7.77 (Pin_77), J8.77 (Pin_77); no longer J1.39 (Pin_39), J2.39 (Pin_39), J3.39 (Pin_39), J4.39 (Pin_39), J5.39 (Pin_39), J6.39 (Pin_39), J7.39 (Pin_39), J8.39 (Pin_39)
- net 4: now also J1.7 (Pin_7), J2.7 (Pin_7), J3.7 (Pin_7), J4.7 (Pin_7), J5.7 (Pin_7), J6.7 (Pin_7), J7.7 (Pin_7), J8.7 (Pin_7); no longer J1.4 (Pin_4), J2.4 (Pin_4), J3.4 (Pin_4), J4.4 (Pin_4), J5.4 (Pin_4), J6.4 (Pin_4), J7.4 (Pin_4), J8.4 (Pin_4)
- net 40: now also J1.79 (Pin_79), J2.79 (Pin_79), J3.79 (Pin_79), J4.79 (Pin_79), J5.79 (Pin_79), J6.79 (Pin_79), J7.79 (Pin_79), J8.79 (Pin_79); no longer J1.40 (Pin_40), J2.40 (Pin_40), J3.40 (Pin_40), J4.40 (Pin_40), J5.40 (Pin_40), J6.40 (Pin_40), J7.40 (Pin_40), J8.40 (Pin_40)
- net 41: now also J1.80 (Pin_80), J2.80 (Pin_80), J3.80 (Pin_80), J4.80 (Pin_80), J5.80 (Pin_80), J6.80 (Pin_80), J7.80 (Pin_80), J8.80 (Pin_80); no longer J1.41 (Pin_41), J2.41 (Pin_41), J3.41 (Pin_41), J4.41 (Pin_41), J5.41 (Pin_41), J6.41 (Pin_41), J7.41 (Pin_41), J8.41 (Pin_41)
- net 42: now also J1.78 (Pin_78), J2.78 (Pin_78), J3.78 (Pin_78), J4.78 (Pin_78), J5.78 (Pin_78), J6.78 (Pin_78), J7.78 (Pin_78), J8.78 (Pin_78); no longer J1.42 (Pin_42), J2.42 (Pin_42), J3.42 (Pin_42), J4.42 (Pin_42), J5.42 (Pin_42), J6.42 (Pin_42), J7.42 (Pin_42), J8.42 (Pin_42)
- net 43: now also J1.76 (Pin_76), J2.76 (Pin_76), J3.76 (Pin_76), J4.76 (Pin_76), J5.76 (Pin_76), J6.76 (Pin_76), J7.76 (Pin_76), J8.76 (Pin_76); no longer J1.43 (Pin_43), J2.43 (Pin_43), J3.43 (Pin_43), J4.43 (Pin_43), J5.43 (Pin_43), J6.43 (Pin_43), J7.43 (Pin_43), J8.43 (Pin_43)
- net 44: now also J1.74 (Pin_74), J2.74 (Pin_74), J3.74 (Pin_74), J4.74 (Pin_74), J5.74 (Pin_74), J6.74 (Pin_74), J7.74 (Pin_74), J8.74 (Pin_74); no longer J1.44 (Pin_44), J2.44 (Pin_44), J3.44 (Pin_44), J4.44 (Pin_44), J5.44 (Pin_44), J6.44 (Pin_44), J7.44 (Pin_44), J8.44 (Pin_44)
- net 45: now also J1.72 (Pin_72), J2.72 (Pin_72), J3.72 (Pin_72), J4.72 (Pin_72), J5.72 (Pin_72), J6.72 (Pin_72), J7.72 (Pin_72), J8.72 (Pin_72); no longer J1.45 (Pin_45), J2.45 (Pin_45), J3.45 (Pin_45), J4.45 (Pin_45), J5.45 (Pin_45), J6.45 (Pin_45), J7.45 (Pin_45), J8.45 (Pin_45)
- net 46: now also J1.70 (Pin_70), J2.70 (Pin_70), J3.70 (Pin_70), J4.70 (Pin_70), J5.70 (Pin_70), J6.70 (Pin_70), J7.70 (Pin_70), J8.70 (Pin_70); no longer J1.46 (Pin_46), J2.46 (Pin_46), J3.46 (Pin_46), J4.46 (Pin_46), J5.46 (Pin_46), J6.46 (Pin_46), J7.46 (Pin_46), J8.46 (Pin_46)
- net 47: now also J1.68 (Pin_68), J2.68 (Pin_68), J3.68 (Pin_68), J4.68 (Pin_68), J5.68 (Pin_68), J6.68 (Pin_68), J7.68 (Pin_68), J8.68 (Pin_68); no longer J1.47 (Pin_47), J2.47 (Pin_47), J3.47 (Pin_47), J4.47 (Pin_47), J5.47 (Pin_47), J6.47 (Pin_47), J7.47 (Pin_47), J8.47 (Pin_47)
- net 48: now also J1.66 (Pin_66), J2.66 (Pin_66), J3.66 (Pin_66), J4.66 (Pin_66), J5.66 (Pin_66), J6.66 (Pin_66), J7.66 (Pin_66), J8.66 (Pin_66); no longer J1.48 (Pin_48), J2.48 (Pin_48), J3.48 (Pin_48), J4.48 (Pin_48), J5.48 (Pin_48), J6.48 (Pin_48), J7.48 (Pin_48), J8.48 (Pin_48)
- net 49: now also J1.64 (Pin_64), J2.64 (Pin_64), J3.64 (Pin_64), J4.64 (Pin_64), J5.64 (Pin_64), J6.64 (Pin_64), J7.64 (Pin_64), J8.64 (Pin_64); no longer J1.49 (Pin_49), J2.49 (Pin_49), J3.49 (Pin_49), J4.49 (Pin_49), J5.49 (Pin_49), J6.49 (Pin_49), J7.49 (Pin_49), J8.49 (Pin_49)
- net 5: now also J1.9 (Pin_9), J2.9 (Pin_9), J3.9 (Pin_9), J4.9 (Pin_9), J5.9 (Pin_9), J6.9 (Pin_9), J7.9 (Pin_9), J8.9 (Pin_9); no longer J1.5 (Pin_5), J2.5 (Pin_5), J3.5 (Pin_5), J4.5 (Pin_5), J5.5 (Pin_5), J6.5 (Pin_5), J7.5 (Pin_5), J8.5 (Pin_5)
- net 50: now also J1.62 (Pin_62), J2.62 (Pin_62), J3.62 (Pin_62), J4.62 (Pin_62), J5.62 (Pin_62), J6.62 (Pin_62), J7.62 (Pin_62), J8.62 (Pin_62); no longer J1.50 (Pin_50), J2.50 (Pin_50), J3.50 (Pin_50), J4.50 (Pin_50), J5.50 (Pin_50), J6.50 (Pin_50), J7.50 (Pin_50), J8.50 (Pin_50)
- net 51: now also J1.60 (Pin_60), J2.60 (Pin_60), J3.60 (Pin_60), J4.60 (Pin_60), J5.60 (Pin_60), J6.60 (Pin_60), J7.60 (Pin_60), J8.60 (Pin_60); no longer J1.51 (Pin_51), J2.51 (Pin_51), J3.51 (Pin_51), J4.51 (Pin_51), J5.51 (Pin_51), J6.51 (Pin_51), J7.51 (Pin_51), J8.51 (Pin_51)
- net 52: now also J1.58 (Pin_58), J2.58 (Pin_58), J3.58 (Pin_58), J4.58 (Pin_58), J5.58 (Pin_58), J6.58 (Pin_58), J7.58 (Pin_58), J8.58 (Pin_58); no longer J1.52 (Pin_52), J2.52 (Pin_52), J3.52 (Pin_52), J4.52 (Pin_52), J5.52 (Pin_52), J6.52 (Pin_52), J7.52 (Pin_52), J8.52 (Pin_52)
- net 53: now also J1.56 (Pin_56), J2.56 (Pin_56), J3.56 (Pin_56), J4.56 (Pin_56), J5.56 (Pin_56), J6.56 (Pin_56), J7.56 (Pin_56), J8.56 (Pin_56); no longer J1.53 (Pin_53), J2.53 (Pin_53), J3.53 (Pin_53), J4.53 (Pin_53), J5.53 (Pin_53), J6.53 (Pin_53), J7.53 (Pin_53), J8.53 (Pin_53)
- net 55: now also J1.52 (Pin_52), J2.52 (Pin_52), J3.52 (Pin_52), J4.52 (Pin_52), J5.52 (Pin_52), J6.52 (Pin_52), J7.52 (Pin_52), J8.52 (Pin_52); no longer J1.55 (Pin_55), J2.55 (Pin_55), J3.55 (Pin_55), J4.55 (Pin_55), J5.55 (Pin_55), J6.55 (Pin_55), J7.55 (Pin_55), J8.55 (Pin_55)
- net 56: now also J1.50 (Pin_50), J2.50 (Pin_50), J3.50 (Pin_50), J4.50 (Pin_50), J5.50 (Pin_50), J6.50 (Pin_50), J7.50 (Pin_50), J8.50 (Pin_50); no longer J1.56 (Pin_56), J2.56 (Pin_56), J3.56 (Pin_56), J4.56 (Pin_56), J5.56 (Pin_56), J6.56 (Pin_56), J7.56 (Pin_56), J8.56 (Pin_56)
- net 57: now also J1.48 (Pin_48), J2.48 (Pin_48), J3.48 (Pin_48), J4.48 (Pin_48), J5.48 (Pin_48), J6.48 (Pin_48), J7.48 (Pin_48), J8.48 (Pin_48); no longer J1.57 (Pin_57), J2.57 (Pin_57), J3.57 (Pin_57), J4.57 (Pin_57), J5.57 (Pin_57), J6.57 (Pin_57), J7.57 (Pin_57), J8.57 (Pin_57)
- net 58: now also J1.46 (Pin_46), J2.46 (Pin_46), J3.46 (Pin_46), J4.46 (Pin_46), J5.46 (Pin_46), J6.46 (Pin_46), J7.46 (Pin_46), J8.46 (Pin_46); no longer J1.58 (Pin_58), J2.58 (Pin_58), J3.58 (Pin_58), J4.58 (Pin_58), J5.58 (Pin_58), J6.58 (Pin_58), J7.58 (Pin_58), J8.58 (Pin_58)
- net 59: now also J1.44 (Pin_44), J2.44 (Pin_44), J3.44 (Pin_44), J4.44 (Pin_44), J5.44 (Pin_44), J6.44 (Pin_44), J7.44 (Pin_44), J8.44 (Pin_44); no longer J1.59 (Pin_59), J2.59 (Pin_59), J3.59 (Pin_59), J4.59 (Pin_59), J5.59 (Pin_59), J6.59 (Pin_59), J7.59 (Pin_59), J8.59 (Pin_59)
- net 6: now also J1.11 (Pin_11), J2.11 (Pin_11), J3.11 (Pin_11), J4.11 (Pin_11), J5.11 (Pin_11), J6.11 (Pin_11), J7.11 (Pin_11), J8.11 (Pin_11); no longer J1.6 (Pin_6), J2.6 (Pin_6), J3.6 (Pin_6), J4.6 (Pin_6), J5.6 (Pin_6), J6.6 (Pin_6), J7.6 (Pin_6), J8.6 (Pin_6)
- net 60: now also J1.42 (Pin_42), J2.42 (Pin_42), J3.42 (Pin_42), J4.42 (Pin_42), J5.42 (Pin_42), J6.42 (Pin_42), J7.42 (Pin_42), J8.42 (Pin_42); no longer J1.60 (Pin_60), J2.60 (Pin_60), J3.60 (Pin_60), J4.60 (Pin_60), J5.60 (Pin_60), J6.60 (Pin_60), J7.60 (Pin_60), J8.60 (Pin_60)
- net 61: now also J1.40 (Pin_40), J2.40 (Pin_40), J3.40 (Pin_40), J4.40 (Pin_40), J5.40 (Pin_40), J6.40 (Pin_40), J7.40 (Pin_40), J8.40 (Pin_40); no longer J1.61 (Pin_61), J2.61 (Pin_61), J3.61 (Pin_61), J4.61 (Pin_61), J5.61 (Pin_61), J6.61 (Pin_61), J7.61 (Pin_61), J8.61 (Pin_61)
- net 62: now also J1.38 (Pin_38), J2.38 (Pin_38), J3.38 (Pin_38), J4.38 (Pin_38), J5.38 (Pin_38), J6.38 (Pin_38), J7.38 (Pin_38), J8.38 (Pin_38); no longer J1.62 (Pin_62), J2.62 (Pin_62), J3.62 (Pin_62), J4.62 (Pin_62), J5.62 (Pin_62), J6.62 (Pin_62), J7.62 (Pin_62), J8.62 (Pin_62)
- net 63: now also J1.36 (Pin_36), J2.36 (Pin_36), J3.36 (Pin_36), J4.36 (Pin_36), J5.36 (Pin_36), J6.36 (Pin_36), J7.36 (Pin_36), J8.36 (Pin_36); no longer J1.63 (Pin_63), J2.63 (Pin_63), J3.63 (Pin_63), J4.63 (Pin_63), J5.63 (Pin_63), J6.63 (Pin_63), J7.63 (Pin_63), J8.63 (Pin_63)
- net 64: now also J1.34 (Pin_34), J2.34 (Pin_34), J3.34 (Pin_34), J4.34 (Pin_34), J5.34 (Pin_34), J6.34 (Pin_34), J7.34 (Pin_34), J8.34 (Pin_34); no longer J1.64 (Pin_64), J2.64 (Pin_64), J3.64 (Pin_64), J4.64 (Pin_64), J5.64 (Pin_64), J6.64 (Pin_64), J7.64 (Pin_64), J8.64 (Pin_64)
- net 65: now also J1.32 (Pin_32), J2.32 (Pin_32), J3.32 (Pin_32), J4.32 (Pin_32), J5.32 (Pin_32), J6.32 (Pin_32), J7.32 (Pin_32), J8.32 (Pin_32); no longer J1.65 (Pin_65), J2.65 (Pin_65), J3.65 (Pin_65), J4.65 (Pin_65), J5.65 (Pin_65), J6.65 (Pin_65), J7.65 (Pin_65), J8.65 (Pin_65)
- net 66: now also J1.30 (Pin_30), J2.30 (Pin_30), J3.30 (Pin_30), J4.30 (Pin_30), J5.30 (Pin_30), J6.30 (Pin_30), J7.30 (Pin_30), J8.30 (Pin_30); no longer J1.66 (Pin_66), J2.66 (Pin_66), J3.66 (Pin_66), J4.66 (Pin_66), J5.66 (Pin_66), J6.66 (Pin_66), J7.66 (Pin_66), J8.66 (Pin_66)
- net 67: now also J1.28 (Pin_28), J2.28 (Pin_28), J3.28 (Pin_28), J4.28 (Pin_28), J5.28 (Pin_28), J6.28 (Pin_28), J7.28 (Pin_28), J8.28 (Pin_28); no longer J1.67 (Pin_67), J2.67 (Pin_67), J3.67 (Pin_67), J4.67 (Pin_67), J5.67 (Pin_67), J6.67 (Pin_67), J7.67 (Pin_67), J8.67 (Pin_67)
- net 68: now also J1.26 (Pin_26), J2.26 (Pin_26), J3.26 (Pin_26), J4.26 (Pin_26), J5.26 (Pin_26), J6.26 (Pin_26), J7.26 (Pin_26), J8.26 (Pin_26); no longer J1.68 (Pin_68), J2.68 (Pin_68), J3.68 (Pin_68), J4.68 (Pin_68), J5.68 (Pin_68), J6.68 (Pin_68), J7.68 (Pin_68), J8.68 (Pin_68)
- net 69: now also J1.24 (Pin_24), J2.24 (Pin_24), J3.24 (Pin_24), J4.24 (Pin_24), J5.24 (Pin_24), J6.24 (Pin_24), J7.24 (Pin_24), J8.24 (Pin_24); no longer J1.69 (Pin_69), J2.69 (Pin_69), J3.69 (Pin_69), J4.69 (Pin_69), J5.69 (Pin_69), J6.69 (Pin_69), J7.69 (Pin_69), J8.69 (Pin_69)
- net 7: now also J1.13 (Pin_13), J2.13 (Pin_13), J3.13 (Pin_13), J4.13 (Pin_13), J5.13 (Pin_13), J6.13 (Pin_13), J7.13 (Pin_13), J8.13 (Pin_13); no longer J1.7 (Pin_7), J2.7 (Pin_7), J3.7 (Pin_7), J4.7 (Pin_7), J5.7 (Pin_7), J6.7 (Pin_7), J7.7 (Pin_7), J8.7 (Pin_7)
- net 70: now also J1.22 (Pin_22), J2.22 (Pin_22), J3.22 (Pin_22), J4.22 (Pin_22), J5.22 (Pin_22), J6.22 (Pin_22), J7.22 (Pin_22), J8.22 (Pin_22); no longer J1.70 (Pin_70), J2.70 (Pin_70), J3.70 (Pin_70), J4.70 (Pin_70), J5.70 (Pin_70), J6.70 (Pin_70), J7.70 (Pin_70), J8.70 (Pin_70)
- net 71: now also J1.20 (Pin_20), J2.20 (Pin_20), J3.20 (Pin_20), J4.20 (Pin_20), J5.20 (Pin_20), J6.20 (Pin_20), J7.20 (Pin_20), J8.20 (Pin_20); no longer J1.71 (Pin_71), J2.71 (Pin_71), J3.71 (Pin_71), J4.71 (Pin_71), J5.71 (Pin_71), J6.71 (Pin_71), J7.71 (Pin_71), J8.71 (Pin_71)
- net 72: now also J1.18 (Pin_18), J2.18 (Pin_18), J3.18 (Pin_18), J4.18 (Pin_18), J5.18 (Pin_18), J6.18 (Pin_18), J7.18 (Pin_18), J8.18 (Pin_18); no longer J1.72 (Pin_72), J2.72 (Pin_72), J3.72 (Pin_72), J4.72 (Pin_72), J5.72 (Pin_72), J6.72 (Pin_72), J7.72 (Pin_72), J8.72 (Pin_72)
- net 73: now also J1.16 (Pin_16), J2.16 (Pin_16), J3.16 (Pin_16), J4.16 (Pin_16), J5.16 (Pin_16), J6.16 (Pin_16), J7.16 (Pin_16), J8.16 (Pin_16); no longer J1.73 (Pin_73), J2.73 (Pin_73), J3.73 (Pin_73), J4.73 (Pin_73), J5.73 (Pin_73), J6.73 (Pin_73), J7.73 (Pin_73), J8.73 (Pin_73)
- net 74: now also J1.14 (Pin_14), J2.14 (Pin_14), J3.14 (Pin_14), J4.14 (Pin_14), J5.14 (Pin_14), J6.14 (Pin_14), J7.14 (Pin_14), J8.14 (Pin_14); no longer J1.74 (Pin_74), J2.74 (Pin_74), J3.74 (Pin_74), J4.74 (Pin_74), J5.74 (Pin_74), J6.74 (Pin_74), J7.74 (Pin_74), J8.74 (Pin_74)
- net 75: now also J1.12 (Pin_12), J2.12 (Pin_12), J3.12 (Pin_12), J4.12 (Pin_12), J5.12 (Pin_12), J6.12 (Pin_12), J7.12 (Pin_12), J8.12 (Pin_12); no longer J1.75 (Pin_75), J2.75 (Pin_75), J3.75 (Pin_75), J4.75 (Pin_75), J5.75 (Pin_75), J6.75 (Pin_75), J7.75 (Pin_75), J8.75 (Pin_75)
- net 76: now also J1.10 (Pin_10), J2.10 (Pin_10), J3.10 (Pin_10), J4.10 (Pin_10), J5.10 (Pin_10), J6.10 (Pin_10), J7.10 (Pin_10), J8.10 (Pin_10); no longer J1.76 (Pin_76), J2.76 (Pin_76), J3.76 (Pin_76), J4.76 (Pin_76), J5.76 (Pin_76), J6.76 (Pin_76), J7.76 (Pin_76), J8.76 (Pin_76)
- net 77: now also J1.8 (Pin_8), J2.8 (Pin_8), J3.8 (Pin_8), J4.8 (Pin_8), J5.8 (Pin_8), J6.8 (Pin_8), J7.8 (Pin_8), J8.8 (Pin_8); no longer J1.77 (Pin_77), J2.77 (Pin_77), J3.77 (Pin_77), J4.77 (Pin_77), J5.77 (Pin_77), J6.77 (Pin_77), J7.77 (Pin_77), J8.77 (Pin_77)
- net 78: now also J1.6 (Pin_6), J2.6 (Pin_6), J3.6 (Pin_6), J4.6 (Pin_6), J5.6 (Pin_6), J6.6 (Pin_6), J7.6 (Pin_6), J8.6 (Pin_6); no longer J1.78 (Pin_78), J2.78 (Pin_78), J3.78 (Pin_78), J4.78 (Pin_78), J5.78 (Pin_78), J6.78 (Pin_78), J7.78 (Pin_78), J8.78 (Pin_78)
- net 79: now also J1.4 (Pin_4), J2.4 (Pin_4), J3.4 (Pin_4), J4.4 (Pin_4), J5.4 (Pin_4), J6.4 (Pin_4), J7.4 (Pin_4), J8.4 (Pin_4); no longer J1.79 (Pin_79), J2.79 (Pin_79), J3.79 (Pin_79), J4.79 (Pin_79), J5.79 (Pin_79), J6.79 (Pin_79), J7.79 (Pin_79), J8.79 (Pin_79)
- net 8: now also J1.15 (Pin_15), J2.15 (Pin_15), J3.15 (Pin_15), J4.15 (Pin_15), J5.15 (Pin_15), J6.15 (Pin_15), J7.15 (Pin_15), J8.15 (Pin_15); no longer J1.8 (Pin_8), J2.8 (Pin_8), J3.8 (Pin_8), J4.8 (Pin_8), J5.8 (Pin_8), J6.8 (Pin_8), J7.8 (Pin_8), J8.8 (Pin_8)
- net 80: now also J1.2 (Pin_2), J2.2 (Pin_2), J3.2 (Pin_2), J4.2 (Pin_2), J5.2 (Pin_2), J6.2 (Pin_2), J7.2 (Pin_2), J8.2 (Pin_2); no longer J1.80 (Pin_80), J2.80 (Pin_80), J3.80 (Pin_80), J4.80 (Pin_80), J5.80 (Pin_80), J6.80 (Pin_80), J7.80 (Pin_80), J8.80 (Pin_80)
- net 9: now also J1.17 (Pin_17), J2.17 (Pin_17), J3.17 (Pin_17), J4.17 (Pin_17), J5.17 (Pin_17), J6.17 (Pin_17), J7.17 (Pin_17), J8.17 (Pin_17); no longer J1.9 (Pin_9), J2.9 (Pin_9), J3.9 (Pin_9), J4.9 (Pin_9), J5.9 (Pin_9), J6.9 (Pin_9), J7.9 (Pin_9), J8.9 (Pin_9)
Changed lines of the file:
@@
 	900  700  1000 800
 $Comp
-L Connector_Generic:Conn_02x40_Counter_Clockwise J1
+L Connector_Generic:Conn_02x40_Odd_Even J1
 U 1 1 60E8A2E4
 P 1300 2700
@@
 	2150 700  2250 800
 $Comp
-L Connector_Generic:Conn_02x40_Counter_Clockwise J2
+L Connector_Generic:Conn_02x40_Odd_Even J2
 U 1 1 60F0B856
 P 2550 2700
@@
 	3350 700  3450 800
 $Comp
-L Connector_Generic:Conn_02x40_Counter_Clockwise J3
+L Connector_Generic:Conn_02x40_Odd_Even J3
 U 1 1 60F251FE
 P 3750 2700
@@
 	4600 700  4700 800
 $Comp
-L Connector_Generic:Conn_02x40_Counter_Clockwise J4
+L Connector_Generic:Conn_02x40_Odd_Even J4
 U 1 1 60F252F8
 P 5000 2700
@@
 	5900 700  6000 800
 $Comp
-L Connector_Generic:Conn_02x40_Counter_Clockwise J5
+L Connector_Generic:Conn_02x40_Odd_Even J5
 U 1 1 60F652B0
 P 6300 2700
@@
 	7150 700  7250 800
 $Comp
-L Connector_Generic:Conn_02x40_Counter_Clockwise J6
+L Connector_Generic:Conn_02x40_Odd_Even J6
 U 1 1 60F653AA
 P 7550 2700
@@
 	8350 700  8450 800
 $Comp
-L Connector_Generic:Conn_02x40_Counter_Clockwise J7
+L Connector_Generic:Conn_02x40_Odd_Even J7
 U 1 1 60F654A4
 P 8750 2700
@@
 	4250 4850 4600 4850
 $Comp
-L Connector_Generic:Conn_02x40_Counter_Clockwise J8
+L Connector_Generic:Conn_02x40_Odd_Even J8
 U 1 1 61AB8D58
 P 10000 2700
